File: Mechaduino02.sch (EAGLE design)
At the start: 64 parts, among them IC1 SAMD21G18A-AUT, Q1 BSS138, Q2 NFET, Q3 BSS138, Q4 BSS138, Q5 BSS138, U1 TLV70233PDBVR, Y1 32,768Khz

Commit message: updated image
Other:
- note added: "0.2"
- note removed: "0.1"
Changed lines of the file:
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@@
 Arduino Zero by Arduino.cc              Arduino M0 by Arduino.org
 Neutrino by Rabidprototypes.com    SAMD21 Dev Breakout by Sparkfun.com</text>
-<text x="426.72" y="12.7" size="2.54" layer="94" align="top-left">0.1</text>
+<text x="426.72" y="12.7" size="2.54" layer="94" align="top-left">0.2</text>
 <text x="134.62" y="266.7" size="1.778" layer="97" rot="R180">Arduino Zero Compatible</text>
 <wire x1="180.34" y1="152.4" x2="294.64" y2="152.4" width="0.2032" layer="97" style="longdash"/>
